File: MidiToCVShield.sch (KiCad schematic (older format))
At the start: 32 parts, among them K1 CONN_3, P1 CONN_2, P10 CONN_1, P11 CONN_1, P2 CONN_2, P3 CONN_2, P4 CONN_2, P5 CONN_2, P6 CONN_2, P7 CONN_2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

Commit message: Version Sent to OSHPark for manufacture
Parts:
- removed Q1: PN2222A, TO92, symbol PN2222A
- added Q1: NPN, symbol NPN
- R2: value R -> 1K
- R3: value R -> 10K
Connections:
- net +5V: now also Q1.3 (C)
- net at P7.2 (GND), P9.1, R9.2: now also D1.2 (K)
- net at R3.2: now also Q1.2 (B)
- net at R2.1: now also Q1.1 (E)
